File: mk19-flex-pcb.kicad_pcb (KiCad board)
At the start: 2 copper layers, 268.4 x 46.9 mm, 13 parts

Commit message: ready for review
Routing:
- net col4: track 0.00 -> 720.7 mm, vias 0 -> 12
- net col3: track 0.00 -> 678.9 mm, vias 0 -> 10
- net col1: track 0.00 -> 647.5 mm, vias 0 -> 10
- net col5: track 0.00 -> 609.3 mm, vias 0 -> 9
- net col2: track 0.00 -> 603.3 mm, vias 0 -> 9
- net row4: track 0.00 -> 593.8 mm, vias 0 -> 7
- net row5: track 0.00 -> 584.8 mm, vias 0 -> 7
- net row6: track 0.00 -> 579.0 mm, vias 0 -> 7
- net row2: track 0.00 -> 539.3 mm, vias 0 -> 7
- net row3: track 0.00 -> 531.4 mm, vias 0 -> 7
- net row1: track 11.5 -> 539.2 mm, vias 0 -> 7
- net row0: track 945.9 -> 962.0 mm, vias 11 -> 15
- net Net-(COL-4-Pin_2): track 84.0 -> 89.6 mm, vias 4 -> 2
- net Net-(COL-4-Pin_11): track 84.5 -> 89.5 mm, vias 4 -> 2
- net Net-(COL-2-Pin_2): track 85.6 -> 90.4 mm, vias 4 -> 2
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Other:
- board size 268.4 x 46.9 mm -> 269.8 x 46.9 mm
